Commit message: add slope

File: src/AMP_for_hardware/resources/robots/jl/urdf/jl.urdf (robot description, URDF)
Before this commit: robot robot, 18 links, 17 joints
Links:
- link FR_calf: geometry collision box size=0.16850767 0.018 0.015; visual mesh filename=../meshes/FR_calf_link.STL scale=1 1 1
Joints:
- joint FL_calf_joint: limit lower=-2.65 upper=-0.9 effort=12.0001 velocity=30.9971 -> lower=-2.55 upper=-0.9 effort=12.0001 velocity=30.9971
- joint FR_calf_joint: limit lower=-2.65 upper=-0.9 effort=12.0001 velocity=30.9971 -> lower=-2.55 upper=-0.9 effort=12.0001 velocity=30.9971
- joint RL_calf_joint: limit lower=-2.65 upper=-0.9 effort=12.0001 velocity=30.9971 -> lower=-2.55 upper=-0.9 effort=12.0001 velocity=30.9971
- joint RR_calf_joint: limit lower=-2.65 upper=-0.9 effort=12.0001 velocity=30.9971 -> lower=-2.55 upper=-0.9 effort=12.0001 velocity=30.9971
